File: Pressure-Sensor-Module.brd (EAGLE design)
At the start: 52.1 x 25.4 mm, 18 parts, among them IC1 ATTINY85

Commit message: v2 Pressure Sensor Board
Parts:
- ICSP: device SparkFun-Connectors:2X3_POGO -> tag-connect:TC2030-MCP-NL-CP
- moved FD2 8.05 mm to (0.89, 1.02)
- moved ICSP 1.05 mm to (35.3, 5.59)
Connections:
- removed net INTPIN: HEADER.P$5, IC1.6, ICSP.P$1
- removed net SENSE: IC1.7, ICSP.P$3, PRESSURE-SENSOR.4
- new net CLK/SENSE: IC1.7, ICSP.5, PRESSURE-SENSOR.4
- new net MISO/INT: HEADER.P$5, IC1.6, ICSP.6
- net GND: now also ICSP.3; no longer ICSP.P$6
- net MOSI/D0: now also ICSP.4; no longer ICSP.P$4
- net RST/D5: now also ICSP.1; no longer ICSP.P$5
- net VCC: now also ICSP.2; no longer ICSP.P$2
Routing:
- net CLK/SENSE: track 0.00 -> 30.6 mm, vias 0 -> 2
- net INTPIN: track 27.4 -> 0.00 mm
- net MISO/INT: track 0.00 -> 26.0 mm
- net SENSE: track 26.0 -> 0.00 mm, vias 1 -> 0
- net RST/D5: track 34.6 -> 42.8 mm
- net VCC: track 42.7 -> 48.6 mm, vias 1 -> 2
- net LED: track 21.2 -> 26.6 mm, vias 0 -> 2
- net !CLEAR!: track 21.8 -> 24.9 mm, vias 1 -> 0
- net !EN!: track 22.0 -> 20.6 mm
- net LED-PWR: track 7.75 -> 8.81 mm
- net MOSI/D0: track 11.2 -> 10.2 mm, vias 1 -> 0
Other:
- outline, holes or cut-outs redrawn
- board text added: "Pressure Sensor Board v2.0 3-15-19"
- board text added: "RST GND CLK"
- board text added: "VCC MOSI MISO"
- board text removed: "MISO CLK RST"
- board text removed: "Pressure Sensor Board v1.1 8-7-18"
- board text removed: "VCC MOSI GND"

Commit message: v2.0 Release Candidate
Parts:
- added C2: 1uF, SparkFun-Capacitors:0805
- added C3: 0.01uF, SparkFun-Capacitors:0805
- added C4: 0.33uF, SparkFun-Capacitors:0805
- added C5, C6: 0.1uF, SparkFun-Capacitors:0805
- added R4, R5: 1k, SparkFun-Resistors:0805
- added R6: 750, SparkFun-Resistors:0805
- ICSP: device tag-connect:TC2030-MCP-NL-CP -> tag-connect:TC2030-MCP-NL
- moved R2 4.71 mm to (41.5, 12.4)
- moved R1 3.71 mm to (25.8, 22.6), turned to 180 degrees
- moved LED1 2.17 mm to (37.2, 12.4)
- moved HEADER 1.76 mm to (37.1, 19.2)
- moved POWER-SWITCH 1.35 mm to (27.1, 18.0)
- moved C1 0.77 mm to (23.6, 8.76)
- moved IC1 0.76 mm to (27.2, 6.35)
- moved R3 0.76 mm to (23.6, 3.81)
Connections:
- removed net VCC-IN: HEADER.P$1, POWER-SWITCH.1, POWER-SWITCH.2, POWER-SWITCH.3, R1.1
- new net +3V3: C6.1, HEADER.P$1, POWER-SWITCH.1, POWER-SWITCH.2, POWER-SWITCH.3, R1.1
- new net INT: HEADER.P$5, R4.2
- new net N$2: HEADER.P$3, R5.2
- new net N$3: PRESSURE-SENSOR.4, R6.2
- net !EN!: now also R5.1; no longer HEADER.P$3
- net CLK/SENSE: now also C4.1, ICSP.3, R6.1; no longer ICSP.5, PRESSURE-SENSOR.4
- net GND: now also C2.2, C3.2, C4.2, C5.2, C6.2, ICSP.6; no longer ICSP.3
- net MISO/INT: now also ICSP.1, R4.1; no longer HEADER.P$5, ICSP.6
- net RST/D5: now also ICSP.5; no longer ICSP.1
- net VCC: now also C2.1, C3.1, C5.1
Routing:
- net VCC-IN: track 15.7 -> 0.00 mm
- net +3V3: track 0.00 -> 13.5 mm
- net INT: track 0.00 -> 12.0 mm
- net LED: track 26.6 -> 14.8 mm
- net !EN!: track 20.6 -> 11.3 mm
- net N$2: track 0.00 -> 6.78 mm
- net LED-PWR: track 8.81 -> 12.9 mm
- net N$3: track 0.00 -> 3.25 mm
- net !CLEAR!: track 24.9 -> 27.8 mm, vias 0 -> 1
- net VCC: track 48.6 -> 50.7 mm, vias 2 -> 0
- net N$1: track 3.43 -> 5.13 mm
- net MOSI/D0: track 10.2 -> 11.4 mm, vias 0 -> 2
- net RST/D5: track 42.8 -> 41.8 mm
- net MISO/INT: track 26.0 -> 25.3 mm
- net CLK/SENSE: track 30.6 -> 31.2 mm, vias 2 -> 0
Other:
- board text added: "MISO CLK !RST"
- board text added: "VCC MOSI GND"
- board text removed: "RST GND CLK"
- board text removed: "VCC MOSI MISO"
